File: hardware/io_revC/io_i2c.kicad_sch (KiCad schematic)
At the start: 24 parts, among them J1 Target Interface, 2716 Pinout, J2 Jumper Block, J3 Jumper Block, Q1 2N7000, U1 2716, U2 74HCT74, U3 74HCT125, U4 74HCT138, U5 74LS04

Commit message: added parallel interface
Parts:
- added C? (x2): 0.1uF, Capacitor_THT:C_Axial_L3.8mm_D2.6mm_P7.50mm_Horizontal, symbol Device:C
- added IC?: MCP23018-E_SP, DIP794W56P254L3486H508Q28N, symbol mouser:MCP23018-E_SP
- added J?: Target Interface, 2716 Pinout, symbol Connector_Generic:Conn_02x12_Counter_Clockwise
- added R?: 10k, Resistor_THT:R_Axial_DIN0207_L6.3mm_D2.5mm_P10.16mm_Horizontal, symbol Device:R
Connections:
- net +5V: now also IC?.11 (VDD), J?.24 (Pin_24), R?.1; no longer U1.21 (VPP), U4.6 (E3)
- net A0: now also IC?.3 (GPB0), J?.8 (Pin_8)
- net A1: now also U1.7 (A1), IC?.4 (GPB1), J?.7 (Pin_7)
- net A10: now also A1.9 (D6), J?.19 (Pin_19)
- net A2: now also IC?.5 (GPB2), J?.6 (Pin_6)
- net A3: now also IC?.6 (GPB3), J?.5 (Pin_5)
- net A4: now also IC?.7 (GPB4), J?.4 (Pin_4)
- net A5: now also IC?.8 (GPB5), J?.3 (Pin_3)
- net A6: now also IC?.9 (GPB6), J?.2 (Pin_2)
- net A7: now also IC?.10 (GPB7), J?.1 (Pin_1)
- net A8: now also A1.7 (D4), J?.23 (Pin_23)
- net A9: now also A1.8 (D5), J?.22 (Pin_22)
- net D0: now also IC?.20 (GPA0), J?.9 (Pin_9)
- net D1: now also IC?.21 (GPA1), J?.10 (Pin_10)
- net D2: now also IC?.22 (GPA2), J?.11 (Pin_11)
- net D3: now also IC?.23 (GPA3), J?.13 (Pin_13)
- net D4: now also IC?.24 (GPA4), J?.14 (Pin_14)
- net D5: now also IC?.25 (GPA5), J?.15 (Pin_15)
- net D6: now also IC?.26 (GPA6), J?.16 (Pin_16)
- net D7: now also IC?.27 (GPA7), J?.17 (Pin_17)
- net GND: now also C?.2, C?.2, IC?.1 (VSS), IC?.15 (ADDR), J?.12 (Pin_12)
- net SCL: now also IC?.12 (SCL)
- net SDA: now also IC?.13 (SDA)
- net program OE: now reaches D1.2 (A), D2.2 (A), D3.2 (A), D4.2 (A), D5.2 (A), D6.2 (A), D7.2 (A), R2.2, U1.20 (~{OE})
- net program OE: now also A1.5 (D2), C?.1
- net Target CE: now reaches J1.18 (~{CE}), J3.1 (Pin_1), U5.5
- net Target CE: now also J?.18 (Pin_18)
- net Target OE: now reaches J1.20 (~{OE}), J3.2 (Pin_2), U5.3
- net Target OE: now also J?.20 (Pin_20)
- net no bypass: now reaches A1.19 (A0)
- net bypass: now reaches A1.20 (A1)
- net no RC: now reaches A1.21 (A2)
- net 138 enable: now reaches A1.22 (A3)
- net 138 enable: now also U4.6 (E3)
- net program WR: now reaches A1.6 (D3)
- net program WR: now also U1.21 (VPP), C?.1
- new net: IC?.16 (~{RESET}), R?.2
- no-connect marks 29 -> 26
Other:
- note added: "TX and RX are used for the serial converter"
- note added: "can program if populated with a 28C16"
- note added: "unhook from target and unhook i2c jumpers when programming"
- moved on the sheet: R2, U2C, U3E, U5G

Commit message: added pulldown for floating fet
Parts:
- added R?: 10k, Resistor_THT:R_Axial_DIN0207_L6.3mm_D2.5mm_P10.16mm_Horizontal, symbol Device:R
Connections:
- net DOUT: now also R?.1
- net GND: now also R?.2
Changed lines of the file:
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@@
     (rev "C")
   )
+  (junction (at 196.85 86.995) (diameter 0) (color 0 0 0 0)
+  )
   (junction (at 178.435 134.62) (diameter 0) (color 0 0 0 0)
   )
@@
   )
   (junction (at 208.28 68.58) (diameter 0) (color 0 0 0 0)
+  )
+  (junction (at 187.96 77.47) (diameter 0) (color 0 0 0 0)
   )
   (junction (at 140.97 58.42) (diameter 0) (color 0 0 0 0)
@@
     (stroke (width 0) (type default) (color 0 0 0 0))
   )
+  (wire (pts (xy 187.96 77.47) (xy 187.96 79.375))
+    (stroke (width 0) (type default) (color 0 0 0 0))
+  )
   (wire (pts (xy 20.32 153.67) (xy 53.34 153.67))
     (stroke (width 0) (type default) (color 0 0 0 0))
@@
     (stroke (width 0) (type default) (color 0 0 0 0))
   )
-  (wire (pts (xy 189.23 80.01) (xy 189.23 95.885))
+  (wire (pts (xy 184.15 80.01) (xy 184.15 95.885))
     (stroke (width 0) (type default) (color 0 0 0 0))
   )
@@
     (stroke (width 0) (type default) (color 0 0 0 0))
   )
+  (wire (pts (xy 187.96 77.47) (xy 189.23 77.47))
+    (stroke (width 0) (type default) (color 0 0 0 0))
+  )
   (wire (pts (xy 38.1 130.81) (xy 35.56 130.81))
     (stroke (width 0) (type default) (color 0 0 0 0))
@@
     (stroke (width 0) (type default) (color 0 0 0 0))
   )
-  (wire (pts (xy 181.61 80.01) (xy 189.23 80.01))
+  (wire (pts (xy 181.61 80.01) (xy 184.15 80.01))
     (stroke (width 0) (type default) (color 0 0 0 0))
   )
@@
     (stroke (width 0) (type default) (color 0 0 0 0))
   )
-  (wire (pts (xy 196.85 82.55) (xy 196.85 88.9))
+  (wire (pts (xy 196.85 82.55) (xy 196.85 86.995))
     (stroke (width 0) (type default) (color 0 0 0 0))
   )
@@
     (stroke (width 0) (type default) (color 0 0 0 0))
   )
+  (wire (pts (xy 187.96 86.995) (xy 196.85 86.995))
+    (stroke (width 0) (type default) (color 0 0 0 0))
+  )
   (wire (pts (xy 201.93 33.02) (xy 201.93 34.29))
     (stroke (width 0) (type default) (color 0 0 0 0))
@@
     (stroke (width 0) (type default) (color 0 0 0 0))
   )
-  (wire (pts (xy 189.23 95.885) (xy 208.28 95.885))
-    (stroke (width 0) (type default) (color 0 0 0 0))
-  )
-  (wire (pts (xy 181.61 77.47) (xy 189.23 77.47))
+  (wire (pts (xy 184.15 95.885) (xy 208.28 95.885))
+    (stroke (width 0) (type default) (color 0 0 0 0))
+  )
+  (wire (pts (xy 181.61 77.47) (xy 187.96 77.47))
     (stroke (width 0) (type default) (color 0 0 0 0))
   )
@@
   )
   (wire (pts (xy 181.61 87.63) (xy 181.61 90.17))
+    (stroke (width 0) (type default) (color 0 0 0 0))
+  )
+  (wire (pts (xy 196.85 86.995) (xy 196.85 88.9))
     (stroke (width 0) (type default) (color 0 0 0 0))
   )
@@
     (pin "1")
   )
+  (symbol (lib_id "Device:R") (at 187.96 83.185 0) (unit 1)
+    (in_bom yes) (on_board yes)
+    (property "Reference" "R?" (id 0) (at 189.738 82.0166 0)
+      (effects (font (size 1.27 1.27)) (justify left))
+    )
+    (property "Value" "10k" (id 1) (at 189.738 84.328 0)
+      (effects (font (size 1.27 1.27)) (justify left))
+    )
+    (property "Footprint" "Resistor_THT:R_Axial_DIN0207_L6.3mm_D2.5mm_P10.16mm_Horizontal" (id 2) (at 186.182 83.185 90)
+      (effects (font (size 1.27 1.27)) hide)
+    )
+    (property "Datasheet" "~" (id 3) (at 187.96 83.185 0)
+      (effects (font (size 1.27 1.27)) hide)
+    )
+    (pin "1")
+    (pin "2")
+  )
   (symbol (lib_id "power:+5V") (at 260.985 144.78 0) (unit 1)
     (in_bom yes) (on_board yes)
@@
       (reference "R?") (unit 1) (value "10k") (footprint "Resistor_THT:R_Axial_DIN0207_L6.3mm_D2.5mm_P10.16mm_Horizontal")
     )
+    (path "/88ce3174-a8b3-4149-886a-872ed4746e98"
+      (reference "R?") (unit 1) (value "10k") (footprint "Resistor_THT:R_Axial_DIN0207_L6.3mm_D2.5mm_P10.16mm_Horizontal")
+    )

Commit message: edited for rev C
Parts:
- removed C?: 0.1uF, Capacitor_THT:C_Axial_L3.8mm_D2.6mm_P7.50mm_Horizontal, symbol Device:C
- added D8, D9: 1N4004, Diode_THT:D_DO-41_SOD81_P2.54mm_Vertical_AnodeUp, symbol Diode:1N4004
- added R3: 1k, Resistor_THT:R_Axial_DIN0207_L6.3mm_D2.5mm_P2.54mm_Vertical, symbol Device:R
- added unit 2 of U3
- added unit 4 of U3
- added unit 3 of U3
- added unit 6 of U5
- added unit 4 of U5
- added unit 5 of U5
- C6: renamed from C?; footprint Capacitor_THT:C_Axial_L3.8mm_D2.6mm_P7.50mm_Horizontal -> Capacitor_SMD:C_0603_1608Metric
- D1, D2, D3, D4, D5, D6, D7: footprint Diode_THT:D_DO-35_SOD27_P7.62mm_Horizontal -> Diode_THT:D_DO-35_SOD27_P2.54mm_Vertical_AnodeUp
- J3: footprint (none) -> Connector_PinHeader_2.54mm:PinHeader_2x03_P2.54mm_Vertical
- J4: renamed from J?; footprint (none) -> Connector_PinHeader_2.54mm:PinHeader_2x12_P2.54mm_Vertical; symbol Connector_Generic:Conn_02x12_Counter_Clockwise -> Connector_Generic:Conn_02x12_Odd_Even
- R1, R2: footprint Resistor_THT:R_Axial_DIN0207_L6.3mm_D2.5mm_P10.16mm_Horizontal -> Resistor_THT:R_Axial_DIN0207_L6.3mm_D2.5mm_P2.54mm_Vertical
- R4, R5: renamed from R?; footprint Resistor_THT:R_Axial_DIN0207_L6.3mm_D2.5mm_P10.16mm_Horizontal -> Resistor_THT:R_Axial_DIN0207_L6.3mm_D2.5mm_P2.54mm_Vertical
- U5: footprint (none) -> Package_DIP:DIP-14_W7.62mm
- U6: renamed from IC?; footprint DIP794W56P254L3486H508Q28N -> Package_DIP:DIP-28_W7.62mm
Connections:
- net +5V: now also D8.1 (K), D9.1 (K), R3.1; no longer J1.24 (VCC), J4.24 (Pin_24)
- net A0: now also J4.15 (Pin_15); no longer J4.8 (Pin_8)
- net A1: now also J4.13 (Pin_13); no longer J4.7 (Pin_7)
- net A10: now also J4.12 (Pin_12); no longer J4.19 (Pin_19)
- net A2: now also J4.11 (Pin_11); no longer J4.6 (Pin_6)
- net A3: now also J4.9 (Pin_9); no longer J4.5 (Pin_5)
- net A4: now also J4.7 (Pin_7); no longer J4.4 (Pin_4)
- net A5: now also J4.5 (Pin_5); no longer J4.3 (Pin_3)
- net A6: now also J4.3 (Pin_3); no longer J4.2 (Pin_2)
- net A8: now also J4.4 (Pin_4); no longer J4.23 (Pin_23)
- net A9: now also J4.6 (Pin_6); no longer J4.22 (Pin_22)
- net D0: now also J4.17 (Pin_17); no longer J4.9 (Pin_9)
- net D1: now also J4.19 (Pin_19); no longer J4.10 (Pin_10)
- net D2: now also J4.21 (Pin_21); no longer J4.11 (Pin_11)
- net D3: now also J4.24 (Pin_24); no longer J4.13 (Pin_13)
- net D4: now also J4.22 (Pin_22); no longer J4.14 (Pin_14)
- net D5: now also J4.20 (Pin_20); no longer J4.15 (Pin_15)
- net D6: now also J4.18 (Pin_18); no longer J4.16 (Pin_16)
- net D7: now also J4.16 (Pin_16); no longer J4.17 (Pin_17)
- net GND: now also J4.23 (Pin_23), U3.10, U3.12, U3.13, U3.9, U5.11, U5.13, U5.9; no longer J4.12 (Pin_12)
- net Target CE: now also J4.14 (Pin_14); no longer J4.18 (Pin_18)
- net Target OE: now also J4.10 (Pin_10); no longer J4.20 (Pin_20)
- net program WR: now also U3.5; no longer U1.21 (VPP)
- net +5VD: now reaches A1.26 (A7)
- net +5VD: now also J1.24 (VCC), J4.2 (Pin_2), D8.2 (A)
- net +5VA: now reaches A1.27 (+5V)
- net +5VA: now also D9.2 (A)
- net VPP: no longer names the net of J1.21 (VPP)
- new net: R3.2, U1.21 (VPP), U3.6
- new net WR enable: U3.4
- no-connect marks 26 -> 25

Commit message: fixed layout a bit and a trace missing, generated gerbers
Connections:
- net WR enable: now also A1.10 (D7)
- no-connect marks 25 -> 24
Changed lines of the file:
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@@
   (no_connect (at 255.27 144.78))
   (no_connect (at 224.79 154.94))
-  (no_connect (at 250.19 77.47))
   (no_connect (at 250.19 85.09))
   (no_connect (at 224.79 59.69))
@@
     (effects (font (size 1.27 1.27)) (justify right bottom))
   )
+  (label "WR enable" (at 250.19 77.47 0)
+    (effects (font (size 1.27 1.27)) (justify left bottom))
+  )
   (label "D3" (at 68.58 66.04 0)
     (effects (font (size 1.27 1.27)) (justify left bottom))
@@
   (symbol (lib_id "power:GND") (at 132.08 161.925 0) (unit 1)
     (in_bom yes) (on_board yes)
-    (property "Reference" "#PWR?" (id 0) (at 132.08 168.275 0)
+    (property "Reference" "#PWR0145" (id 0) (at 132.08 168.275 0)
       (effects (font (size 1.27 1.27)) hide)
     )
@@
   (symbol (lib_id "power:GND") (at 121.285 190.5 0) (unit 1)
     (in_bom yes) (on_board yes)
-    (property "Reference" "#PWR?" (id 0) (at 121.285 196.85 0)
+    (property "Reference" "#PWR0143" (id 0) (at 121.285 196.85 0)
       (effects (font (size 1.27 1.27)) hide)
     )
@@
   (symbol (lib_id "power:GND") (at 129.54 175.26 0) (unit 1)
     (in_bom yes) (on_board yes)
-    (property "Reference" "#PWR?" (id 0) (at 129.54 181.61 0)
+    (property "Reference" "#PWR0144" (id 0) (at 129.54 181.61 0)
       (effects (font (size 1.27 1.27)) hide)
     )
@@
       (reference "#PWR0142") (unit 1) (value "GND") (footprint "")
     )
+    (path "/d44040e4-88a9-4fd1-98c2-f53c3d35a49a"
+      (reference "#PWR0143") (unit 1) (value "GND") (footprint "")
+    )
+    (path "/d69f48b9-a7de-4725-98ab-1310b5582803"
+      (reference "#PWR0144") (unit 1) (value "GND") (footprint "")
+    )
     (path "/425421d5-af6f-4283-942c-b131828f6dd6"
-      (reference "#PWR?") (unit 1) (value "GND") (footprint "")
-    )
-    (path "/d44040e4-88a9-4fd1-98c2-f53c3d35a49a"
-      (reference "#PWR?") (unit 1) (value "GND") (footprint "")
-    )
-    (path "/d69f48b9-a7de-4725-98ab-1310b5582803"
-      (reference "#PWR?") (unit 1) (value "GND") (footprint "")
+      (reference "#PWR0145") (unit 1) (value "GND") (footprint "")
     )
     (path "/00000000-0000-0000-0000-000060a79c85"
