File: hardware/io_revD/_autosave-io_i2c.kicad_sch (KiCad schematic)
At the start: 49 parts, among them J1 Target Interface, 2716 Pinout, J2 Jumper Block, J3 Jumper Block, J4 Target Interface, 2716 Pinout, Q1 2N7000, U1 2716, U2 74HCT74, U3 74HCT125, U4 74HCT138, U6 MCP23018-E_SP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

Commit message: revised schematic
Other:
- note added: "Read from arduino"
- note added: "Write to arduino"
- note removed: "Read"
- note removed: "Write"
Changed lines of the file:
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@@
     (effects (font (size 1.27 1.27)) (justify left bottom))
   )
-  (text "Read" (at 202.565 236.855 0)
+  (text "Read from arduino" (at 202.565 236.855 0)
     (effects (font (size 1.27 1.27)) (justify left bottom))
   )
@@
     (effects (font (size 1.27 1.27)) (justify left bottom))
   )
-  (text "Write" (at 202.565 243.205 0)
+  (text "Write to arduino" (at 202.565 243.205 0)
     (effects (font (size 1.27 1.27)) (justify left bottom))
   )
