File: hardware/io_revD/_autosave-io_i2c.kicad_sch (KiCad schematic)
At the start: 54 parts, among them J1 Target Interface, 2716 Pinout, J10 Conn_01x01, J11 Conn_01x01, J2 Jumper Block, J3 Jumper Block, J4 Target Interface, 2716 Pinout, J5 Conn_01x01, J6 Conn_01x01, J7 Conn_01x01, J8 Conn_01x01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

Commit message: revD board
Parts:
- gave numbers to parts that had none: 4
Changed lines of the file:
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@@
   (symbol (lib_id "Connector_Generic:Conn_01x01") (at 207.645 46.99 270) (unit 1)
     (in_bom yes) (on_board yes)
-    (property "Reference" "J?" (id 0) (at 207.645 50.165 0))
+    (property "Reference" "J12" (id 0) (at 207.645 50.165 0))
     (property "Value" "Conn_01x01" (id 1) (at 205.1836 46.99 0)
       (effects (font (size 1.27 1.27)) hide)
@@
   (symbol (lib_id "Connector_Generic:Conn_01x01") (at 219.71 57.15 90) (unit 1)
     (in_bom yes) (on_board yes)
-    (property "Reference" "J?" (id 0) (at 219.71 53.975 0))
+    (property "Reference" "J14" (id 0) (at 219.71 53.975 0))
     (property "Value" "Conn_01x01" (id 1) (at 222.1714 57.15 0)
       (effects (font (size 1.27 1.27)) hide)
@@
   (symbol (lib_id "Connector_Generic:Conn_01x01") (at 222.885 46.99 270) (unit 1)
     (in_bom yes) (on_board yes)
-    (property "Reference" "J?" (id 0) (at 222.885 50.165 0))
+    (property "Reference" "J15" (id 0) (at 222.885 50.165 0))
     (property "Value" "Conn_01x01" (id 1) (at 220.4236 46.99 0)
       (effects (font (size 1.27 1.27)) hide)
@@
   (symbol (lib_id "power:GND") (at 219.71 62.23 0) (unit 1)
     (in_bom yes) (on_board yes)
-    (property "Reference" "#PWR?" (id 0) (at 219.71 68.58 0)
+    (property "Reference" "#PWR012" (id 0) (at 219.71 68.58 0)
       (effects (font (size 1.27 1.27)) hide)
     )
@@
   (symbol (lib_id "Connector_Generic:Conn_01x01") (at 215.265 46.99 270) (unit 1)
     (in_bom yes) (on_board yes)
-    (property "Reference" "J?" (id 0) (at 215.265 50.165 0))
+    (property "Reference" "J13" (id 0) (at 215.265 50.165 0))
     (property "Value" "Conn_01x01" (id 1) (at 212.8036 46.99 0)
       (effects (font (size 1.27 1.27)) hide)
@@
       (reference "#PWR011") (unit 1) (value "GND") (footprint "")
     )
+    (path "/c5a01f98-82aa-4185-bc9d-ae400d2c132b"
+      (reference "#PWR012") (unit 1) (value "GND") (footprint "")
+    )
     (path "/00000000-0000-0000-0000-00005e291dad"
       (reference "#PWR0101") (unit 1) (value "GND") (footprint "")
@@
       (reference "#PWR0138") (unit 1) (value "+5VD") (footprint "")
     )
-    (path "/c5a01f98-82aa-4185-bc9d-ae400d2c132b"
-      (reference "#PWR?") (unit 1) (value "GND") (footprint "")
-    )
     (path "/00000000-0000-0000-0000-000060a79c85"
       (reference "A1") (unit 1) (value "Arduino_Nano_v3.x") (footprint "Module:Arduino_Nano")
@@
     )
     (path "/19b1efdb-a9fc-4b47-8244-e1fc60c95fb0"
-      (reference "J?") (unit 1) (value "Conn_01x01") (footprint "Connector_PinHeader_2.54mm:PinHeader_1x01_P2.54mm_Vertical")
+      (reference "J12") (unit 1) (value "Conn_01x01") (footprint "Connector_PinHeader_2.54mm:PinHeader_1x01_P2.54mm_Vertical")
+    )
+    (path "/cb4f2bdf-6be5-4993-afae-ec4e7ba25b92"
+      (reference "J13") (unit 1) (value "Conn_01x01") (footprint "Connector_PinHeader_2.54mm:PinHeader_1x01_P2.54mm_Vertical")
     )
     (path "/3584ed87-cd32-43fa-aa55-b11fe8451b01"
-      (reference "J?") (unit 1) (value "Conn_01x01") (footprint "Connector_PinHeader_2.54mm:PinHeader_1x01_P2.54mm_Vertical")
+      (reference "J14") (unit 1) (value "Conn_01x01") (footprint "Connector_PinHeader_2.54mm:PinHeader_1x01_P2.54mm_Vertical")
     )
     (path "/8f994a63-5979-4697-8788-8880d7fb143c"
-      (reference "J?") (unit 1) (value "Conn_01x01") (footprint "Connector_PinHeader_2.54mm:PinHeader_1x01_P2.54mm_Vertical")
-    )
-    (path "/cb4f2bdf-6be5-4993-afae-ec4e7ba25b92"
-      (reference "J?") (unit 1) (value "Conn_01x01") (footprint "Connector_PinHeader_2.54mm:PinHeader_1x01_P2.54mm_Vertical")
+      (reference "J15") (unit 1) (value "Conn_01x01") (footprint "Connector_PinHeader_2.54mm:PinHeader_1x01_P2.54mm_Vertical")
     )
     (path "/00000000-0000-0000-0000-000060a18a27"
