File: hardware/io_revD/io_i2c.kicad_pcb (KiCad board)
At the start: 2 copper layers, 103.6 x 74.9 mm, 61 parts, among them J1 extra CS, J12 Conn_01x01, J13 Conn_01x01, J14 Conn_01x01, J15 Conn_01x01, J16 Target Interface, 2716 Pinout, J2 Jumper Block, J3 Jumper Block, J4 Target Interface, 2716 Pinout, J5 read region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

Commit message: moved to rev E and updated
Changed lines of the file:
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@@
     (property "Sheetname" "")
     (attr through_hole)
-    (fp_text reference "R10" (at 5.109 -0.254 90) (layer "F.SilkS")
+    (fp_text reference "R10" (at 5.109 -0.254 -90 unlocked) (layer "F.SilkS")
       (effects (font (size 1 1) (thickness 0.15)))
     )
-    (fp_text value "4.7k" (at -3.273 -0.254 90) (layer "F.SilkS")
+    (fp_text value "4.7k" (at -3.273 -0.254 -90 unlocked) (layer "F.SilkS")
       (effects (font (size 1 1) (thickness 0.15)))
     )
