File: hardware/io_revE/io_i2c.kicad_sch (KiCad schematic)
At the start: 55 parts, among them J1 extra CS, J12 Conn_01x01, J13 Conn_01x01, J14 Conn_01x01, J15 Conn_01x01, J16 Target Interface, 2716 Pinout, J2 Jumper Block, J3 Jumper Block, J4 Target Interface, 2716 Pinout, J5 read region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

Commit message: moved to rev E and updated
Parts:
- removed R?: 4.7k, Resistor_THT:R_Axial_DIN0207_L6.3mm_D2.5mm_P2.54mm_Vertical, symbol Device:R
- added R10: 4.7k, Resistor_THT:R_Axial_DIN0207_L6.3mm_D2.5mm_P2.54mm_Vertical, symbol Device:R
Connections:
- net +5V: now also R10.1
- net at J5.3 (Pin_3), U3.1: now also R10.2
Changed lines of the file:
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@@
     (title "Demon Debugger ROM-IO Interface - I2C Version")
     (date "2022-02-27")
-    (rev "E")
+    (rev "D")
   )
   (junction (at 180.975 220.98) (diameter 0) (color 0 0 0 0)
@@
   (junction (at 232.41 85.725) (diameter 0) (color 0 0 0 0)
   )
-  (junction (at 187.325 138.43) (diameter 0) (color 0 0 0 0)
-  )
   (junction (at 185.42 66.675) (diameter 0) (color 0 0 0 0)
   )
@@
   (junction (at 151.13 191.135) (diameter 0) (color 0 0 0 0)
   )
+  (junction (at 187.325 149.86) (diameter 0) (color 0 0 0 0)
+  )
   (junction (at 162.56 66.675) (diameter 0) (color 0 0 0 0)
   )
@@
     (stroke (width 0) (type default) (color 0 0 0 0))
   )
+  (wire (pts (xy 187.325 149.86) (xy 193.04 149.86))
+    (stroke (width 0) (type default) (color 0 0 0 0))
+  )
   (wire (pts (xy 241.3 76.835) (xy 241.3 80.645))
     (stroke (width 0) (type default) (color 0 0 0 0))
@@
     (stroke (width 0) (type default) (color 0 0 0 0))
   )
-  (wire (pts (xy 187.325 138.43) (xy 187.325 245.745))
-    (stroke (width 0) (type default) (color 0 0 0 0))
-  )
   (wire (pts (xy 226.06 83.185) (xy 233.68 83.185))
     (stroke (width 0) (type default) (color 0 0 0 0))
@@
     (stroke (width 0) (type default) (color 0 0 0 0))
   )
+  (wire (pts (xy 187.325 149.86) (xy 187.325 245.745))
+    (stroke (width 0) (type default) (color 0 0 0 0))
+  )
   (wire (pts (xy 151.13 163.83) (xy 151.13 170.815))
     (stroke (width 0) (type default) (color 0 0 0 0))
@@
     (stroke (width 0) (type default) (color 0 0 0 0))
   )
-  (wire (pts (xy 187.325 121.285) (xy 187.325 138.43))
+  (wire (pts (xy 187.325 121.285) (xy 187.325 149.86))
     (stroke (width 0) (type default) (color 0 0 0 0))
   )
@@
     (stroke (width 0) (type default) (color 0 0 0 0))
   )
-  (wire (pts (xy 191.77 138.43) (xy 187.325 138.43))
-    (stroke (width 0) (type default) (color 0 0 0 0))
-  )
   (wire (pts (xy 151.13 170.815) (xy 151.13 175.895))
     (stroke (width 0) (type default) (color 0 0 0 0))
@@
     (pin "1")
   )
-  (symbol (lib_id "power:+5V") (at 191.77 130.81 0) (unit 1)
-    (in_bom yes) (on_board yes)
-    (property "Reference" "#PWR?" (id 0) (at 191.77 134.62 0)
-      (effects (font (size 1.27 1.27)) hide)
-    )
-    (property "Value" "+5V" (id 1) (at 192.151 126.4158 0))
-    (property "Footprint" "" (id 2) (at 191.77 130.81 0)
-      (effects (font (size 1.27 1.27)) hide)
-    )
-    (property "Datasheet" "" (id 3) (at 191.77 130.81 0)
-      (effects (font (size 1.27 1.27)) hide)
-    )
-    (pin "1")
-  )
   (symbol (lib_id "power:+5VD") (at 394.335 224.155 0) (unit 1)
     (in_bom yes) (on_board yes) (fields_autoplaced)
@@
     (pin "9")
   )
+  (symbol (lib_id "power:+5V") (at 193.04 142.24 0) (unit 1)
+    (in_bom yes) (on_board yes)
+    (property "Reference" "#PWR0140" (id 0) (at 193.04 146.05 0)
+      (effects (font (size 1.27 1.27)) hide)
+    )
+    (property "Value" "+5V" (id 1) (at 193.421 137.8458 0))
+    (property "Footprint" "" (id 2) (at 193.04 142.24 0)
+      (effects (font (size 1.27 1.27)) hide)
+    )
+    (property "Datasheet" "" (id 3) (at 193.04 142.24 0)
+      (effects (font (size 1.27 1.27)) hide)
+    )
+    (pin "1")
+  )
   (symbol (lib_id "Device:R") (at 299.085 157.48 0) (unit 1)
     (in_bom yes) (on_board yes)
@@
     (pin "2")
   )
-  (symbol (lib_id "Device:R") (at 191.77 134.62 0) (unit 1)
-    (in_bom yes) (on_board yes)
-    (property "Reference" "R?" (id 0) (at 193.548 133.4516 0)
-      (effects (font (size 1.27 1.27)) (justify left))
-    )
-    (property "Value" "4.7k" (id 1) (at 193.548 135.763 0)
-      (effects (font (size 1.27 1.27)) (justify left))
-    )
-    (property "Footprint" "Resistor_THT:R_Axial_DIN0207_L6.3mm_D2.5mm_P2.54mm_Vertical" (id 2) (at 189.992 134.62 90)
-      (effects (font (size 1.27 1.27)) hide)
-    )
-    (property "Datasheet" "~" (id 3) (at 191.77 134.62 0)
-      (effects (font (size 1.27 1.27)) hide)
-    )
-    (pin "1")
-    (pin "2")
-  )
   (symbol (lib_id "power:+5V") (at 126.365 228.6 0) (unit 1)
     (in_bom yes) (on_board yes)
@@
     (pin "9")
   )
+  (symbol (lib_id "Device:R") (at 193.04 146.05 0) (unit 1)
+    (in_bom yes) (on_board yes)
+    (property "Reference" "R10" (id 0) (at 194.818 144.8816 0)
+      (effects (font (size 1.27 1.27)) (justify left))
+    )
+    (property "Value" "4.7k" (id 1) (at 194.818 147.193 0)
+      (effects (font (size 1.27 1.27)) (justify left))
+    )
+    (property "Footprint" "Resistor_THT:R_Axial_DIN0207_L6.3mm_D2.5mm_P2.54mm_Vertical" (id 2) (at 191.262 146.05 90)
+      (effects (font (size 1.27 1.27)) hide)
+    )
+    (property "Datasheet" "~" (id 3) (at 193.04 146.05 0)
+      (effects (font (size 1.27 1.27)) hide)
+    )
+    (pin "1")
+    (pin "2")
+  )
   (symbol (lib_id "Connector_Generic:Conn_01x01") (at 43.815 87.63 270) (unit 1)
     (in_bom yes) (on_board yes)
@@
       (reference "#PWR0139") (unit 1) (value "+5V") (footprint "")
     )
-    (path "/0b15c878-aeb6-49de-938e-c3b42059a5b7"
-      (reference "#PWR?") (unit 1) (value "+5V") (footprint "")
+    (path "/1593efeb-4759-429e-87bc-982a1c6a8eb7"
+      (reference "#PWR0140") (unit 1) (value "+5V") (footprint "")
     )
     (path "/00000000-0000-0000-0000-000060a79c85"
@@
       (reference "R9") (unit 1) (value "4.7k") (footprint "Resistor_THT:R_Axial_DIN0207_L6.3mm_D2.5mm_P2.54mm_Vertical")
     )
-    (path "/6385d3ec-1c45-400a-99d5-e4d68304bab8"
-      (reference "R?") (unit 1) (value "4.7k") (footprint "Resistor_THT:R_Axial_DIN0207_L6.3mm_D2.5mm_P2.54mm_Vertical")
+    (path "/b60fd6a2-03e4-4281-8b9d-040b4b583c0d"
+      (reference "R10") (unit 1) (value "4.7k") (footprint "Resistor_THT:R_Axial_DIN0207_L6.3mm_D2.5mm_P2.54mm_Vertical")
     )
     (path "/00000000-0000-0000-0000-0000607df9f3"

Commit message: rev e complete overhaul of decoding logic, includes one of 2 possible glitch eliminator circuits
Parts:
- removed D10, D11, D12, D13, D14, D15, D16, D17, D18, D19, D3, D4, D5, D6, D7, D8, D9: 1N4148, Diode_THT:D_DO-35_SOD27_P2.54mm_Vertical_KathodeUp, symbol Diode:1N4148
- removed J1: extra CS, Connector_PinHeader_2.54mm:PinHeader_1x03_P2.54mm_Vertical, symbol Connector_Generic:Conn_01x03
- removed J3: Jumper Block, Connector_PinHeader_2.54mm:PinHeader_2x03_P2.54mm_Vertical, symbol Connector_Generic:Conn_02x03_Odd_Even
- removed J5: read region, Connector_PinHeader_2.54mm:PinHeader_1x03_P2.54mm_Vertical, symbol Connector_Generic:Conn_01x03
- removed J6, J7, J8: Conn_01x01, Connector_PinHeader_2.54mm:PinHeader_1x01_P2.54mm_Vertical, symbol Connector_Generic:Conn_01x01
- removed R10, R2, R3, R9: 4.7k, Resistor_THT:R_Axial_DIN0207_L6.3mm_D2.5mm_P2.54mm_Vertical, symbol Device:R
- removed R7: 1k, Resistor_THT:R_Axial_DIN0207_L6.3mm_D2.5mm_P2.54mm_Vertical, symbol Device:R
- removed U3: 74LS125, Package_DIP:DIP-14_W7.62mm, symbol 74xx:74LS125
- removed U4, U7: 74LS138, Package_DIP:DIP-16_W7.62mm, symbol 74xx:74LS138
- added C? (x2): 0.1uF, Capacitor_THT:C_Axial_L3.8mm_D2.6mm_P7.50mm_Horizontal, symbol Device:C
- added J?: read region, Connector_PinHeader_2.54mm:PinHeader_1x03_P2.54mm_Vertical, symbol Connector_Generic:Conn_01x03
- added J? (x2): Conn_01x01, symbol Connector_Generic:Conn_01x01
- added U? (x4): 74LS30, symbol 74xx:74LS30
- added U? (x5): 74LS02, symbol 74xx:74LS02
- added U? (x7): 74LS04, symbol 74xx:74LS04
- added U?: 74LS138, Package_DIP:DIP-16_W7.62mm, symbol 74xx:74LS138
- added U?: 74LS257, symbol 74xx:74LS257
Connections:
- net Target OE is gone; now on net Target /OE: J16.20 (~{OE}), J4.10 (Pin_10)
- net arduino control CS is gone; now on net Target /CE: A1.22 (A3)
- net +5V: now also C?.1, C?.1, J?.3 (Pin_3), U?.1, U?.14 (VCC), U?.14 (VCC), U?.14 (VCC), U?.14 (VCC), U?.16 (VCC), U?.16 (VCC)
- net A10: now also U?.12, U?.12
- net A5: now also U?.3, U?.9
- net A6: now also U?.11, U?.4
- net A7: now also U?.5, U?.5
- net A8: now also U?.6, U?.6
- net A9: now also U?.11, U?.11
- net D0: now also U?.4 (Za); no longer U1.9 (D0), U6.20 (GPA0)
- net GND: now also C?.2, C?.2, J?.1 (Pin_1), U?.7 (GND), U?.7 (GND), U?.7 (GND), U?.7 (GND), U?.8 (GND), U?.8 (GND)
- net SDA: now also J2.5 (Pin_5), U?.2 (I0a); no longer A1.23 (A4), J2.6 (Pin_6), Q1.3 (D), R1.2
- net 2816/OE: now reaches U1.20 (~{OE})
- net 2816/OE: now also U?.12, U?.15 (OE)
- net /WRITEARD: now reaches U2.11 (C), U2.3 (C)
- net /WRITEARD: now also U?.2
- net Target /OE: now reaches A1.10 (D7)
- net Target /OE: now also U?.2
- net Target CE renamed Target /CE
- net Target /CE: now also U?.3
- new net: A1.23 (A4), J2.6 (Pin_6), Q1.3 (D), R1.2
- new net: J?.2 (Pin_2), U?.1
- new net: U?.10, U?.4
- new net: J?.1 (Pin_1), J?.1 (Pin_1), U?.8, U?.8, U?.9
- new net: U?.11, U?.5, U?.8
- new net: U?.12, U?.4
- new net: U?.1, U?.13
- new net: U?.3, U?.6
- new net: U?.10, U?.5, U?.6
- new net: U?.3, U?.8
- new net FLASHD0: U1.9 (D0), U6.20 (GPA0), U?.3 (I1a)
- new net ROME: U?.1, U?.13, U?.2, U?.2
- new net /READARD: U?.1 (S), U?.4
- no-connect marks 25 -> 24
Other:
- note added: "SDA"
- note added: "To use roms with multiple/interesting chip selects: you can drive both target /ce and target /oe together with one output of a '138 The output of the 138 you use depends on how many of each polarity chip select you need you can use up to 4 positive enables and 2 ngative or, up to 5 negative enables and one positive"
- note added: "high for i2c low for emulate whole rom"
- note added: "use 74ls04 or 74ls14 depending"
- note removed: "0000-00FF"
- note removed: "0100-01FF"
- note removed: "0200-02FF"
- note removed: "0300-03FF"
- note removed: "0400-04FF"
- note removed: "0500-05FF"
- note removed: "0600-06FF"
- note removed: "0700-071F"
- note removed: "0720-073F"
- note removed: "0740-075F"
- note removed: "0760-077F"
- note removed: "0780-079F"
- note removed: "07A0-07BF"
- note removed: "07C0-07DF"
- note removed: "07E0-07FF"
- note removed: "256 byte sections"
- note removed: "32 byte sections"
- note removed: "Read from arduino"
- note removed: "Write to arduino"
- moved on the sheet: R5, U2C
