File: hardware/io_revE/io_i2c.kicad_sch (KiCad schematic)
At the start: 47 parts, among them J12 Conn_01x01, J13 Conn_01x01, J14 Conn_01x01, J15 Conn_01x01, J16 Target Interface, 2716 Pinout, J2 Jumper Block, J4 Target Interface, 2716 Pinout, Q1 2N7000, U1 2716, U2 74LS74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

Commit message: added CS multiplexer for use with rev E board, finished rev E layout
Parts:
- removed C?: 0.1uF, Capacitor_THT:C_Axial_L3.8mm_D2.6mm_P7.50mm_Horizontal, symbol Device:C
- removed U?: 74LS138, Package_DIP:DIP-16_W7.62mm, symbol 74xx:74LS138
- added J6: Conn_01x01, Connector_PinHeader_2.54mm:PinHeader_1x01_P2.54mm_Vertical, symbol Connector_Generic:Conn_01x01
- J3, J5: renamed from J?; footprint (none) -> Connector_PinHeader_2.54mm:PinHeader_1x01_P2.54mm_Vertical
- U4, U5, U7, U8: renamed from U?; footprint (none) -> Package_DIP:DIP-14_W7.62mm
- U9: renamed from U?; footprint (none) -> Package_DIP:DIP-16_W7.62mm
- gave numbers to parts that had none: 2
Connections:
- net A10: now also U7.11; no longer U7.12
- net A7: now also U7.3; no longer U7.5
- net A8: now also U7.5, U8.4; no longer U7.6, U8.6
- net A9: now also U7.12; no longer U7.11
- net GND: now also J6.1 (Pin_1)
- net ROME: now also U8.6; no longer U8.2
- net Target /CE: no longer J4.14 (Pin_14)
- net Target /OE: no longer J4.10 (Pin_10)
- net at U5.10: now also U8.2; no longer U8.4
- net at U5.8: now also U7.6; no longer U7.3
- net program OE: no longer names the net of A1.5 (D2)
- new net Target CE: J4.14 (Pin_14)
- new net Target OE: J4.10 (Pin_10)
- no-connect marks 24 -> 34
Other:
- note removed: "To use roms with multiple/interesting chip selects: you can drive both target /ce and target /oe together with one output of a '138 The output of the 138 you use depends on how many of each polarity chip select you need you can use up to 4 positive enables and 2 ngative or, up to 5 negative enables and one positive"
- moved on the sheet: U5D
