File: hardware/io_revE/io_i2c.kicad_sch (KiCad schematic)
At the start: 34 parts, among them J1 read region, J12 Conn_01x01, J13 Conn_01x01, J14 Conn_01x01, J15 Conn_01x01, J16 Target Interface, 2716 Pinout, J2 Jumper Block, J3 Conn_01x01, J4 Target Interface, 2716 Pinout, J5 Conn_01x01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

Commit message: added gerbers
Connections:
- net Target CE is gone; now on net Target /CE: J4.14 (Pin_14)
- net Target OE is gone; now on net Target /OE: J4.10 (Pin_10)
Changed lines of the file:
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@@
+    (stroke (width 0) (type default) (color 0 0 0 0))
+  )
+  (wire (pts (xy 135.89 46.355) (xy 132.08 46.355))
     (stroke (width 0) (type default) (color 0 0 0 0))
   )
@@
   )
   (wire (pts (xy 132.08 31.115) (xy 142.875 31.115))
+    (stroke (width 0) (type default) (color 0 0 0 0))
+  )
+  (wire (pts (xy 135.89 41.275) (xy 132.08 41.275))
     (stroke (width 0) (type default) (color 0 0 0 0))
   )
@@
     (effects (font (size 1.27 1.27)) (justify right bottom))
   )
-  (label "Target CE" (at 132.08 46.355 0)
-    (effects (font (size 1.27 1.27)) (justify left bottom))
-  )
   (label "program WR" (at 123.19 104.775 180)
     (effects (font (size 1.27 1.27)) (justify right bottom))
@@
   )
   (label "D2" (at 113.03 71.755 0)
-    (effects (font (size 1.27 1.27)) (justify left bottom))
-  )
-  (label "Target OE" (at 132.08 41.275 0)
     (effects (font (size 1.27 1.27)) (justify left bottom))
   )
@@
     )
   )
+  (global_label "Target {slash}OE" (shape input) (at 135.89 41.275 0) (fields_autoplaced)
+    (effects (font (size 1.27 1.27)) (justify left))
+    (property "Intersheet References" "${INTERSHEET_REFS}" (id 0) (at 148.858 41.3544 0)
+      (effects (font (size 1.27 1.27)) (justify left) hide)
+    )
+  )
+  (global_label "Target {slash}CE" (shape input) (at 135.89 46.355 0) (fields_autoplaced)
+    (effects (font (size 1.27 1.27)) (justify left))
+    (property "Intersheet References" "${INTERSHEET_REFS}" (id 0) (at 148.7975 46.4344 0)
+      (effects (font (size 1.27 1.27)) (justify left) hide)
+    )
+  )
