File: hardware/io_revE/io_i2c.kicad_pcb (KiCad board)
At the start: 2 copper layers, 103.6 x 74.9 mm, 60 parts, among them J1 extra CS, J12 Conn_01x01, J13 Conn_01x01, J14 Conn_01x01, J15 Conn_01x01, J16 Target Interface, 2716 Pinout, J2 Jumper Block, J3 Jumper Block, J4 Target Interface, 2716 Pinout, J5 read region, J6 Conn_01x01, J7 Conn_01x01, J8 Conn_01x01, Q1 2N7000, U1 2716, U2 74HCT74, U3 74HCT125, U4 74HCT138, U6 MCP23018-E_SP, U7 74HCT138

Commit message: moved to rev E and updated
Parts:
- added R10: 4.7k, Resistor_THT:R_Axial_DIN0207_L6.3mm_D2.5mm_P2.54mm_Vertical, F.Cu at (135.9, 155.7)
- U2: value 74HCT74 -> 74LS74
- U3: value 74HCT125 -> 74LS125
- U4, U7: value 74HCT138 -> 74LS138
- moved R7 0.34 mm to (139.2, 155.7)
Routing:
- net Net-(J5-Pad3): track 93.5 -> 102.1 mm, vias 2 -> 3
- net +5V: track 278.1 -> 280.9 mm
- net Net-(D10-Pad2): track 107.0 -> 108.3 mm
Other:
- board text added: "Demon Debugger Rev. E Knarfian Labs Frank Palazzolo Evan Allen"
- board text removed: "Demon Debugger Rev. D Knarfian Labs Frank Palazzolo Evan Allen"
Changed lines of the file:
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@@
       (effects (font (size 1 1) (thickness 0.15)))
     )
-    (fp_text value "74HCT138" (at 3.81 11.176 180) (layer "F.SilkS")
+    (fp_text value "74LS138" (at 3.81 11.176 180) (layer "F.SilkS")
       (effects (font (size 1 1) (thickness 0.15)))
     )
@@
   )
   (footprint "Resistor_THT:R_Axial_DIN0207_L6.3mm_D2.5mm_P2.54mm_Vertical" (layer "F.Cu")
+    (at 135.89 155.673 -90)
+    (descr "Resistor, Axial_DIN0207 series, Axial, Vertical, pin pitch=2.54mm, 0.25W = 1/4W, length*diameter=6.3*2.5mm^2, http://cdn-reichelt.de/documents/datenblatt/B400/1_4W%23YAG.pdf")
+    (tags "Resistor Axial_DIN0207 series Axial Vertical pin pitch 2.54mm 0.25W = 1/4W length 6.3mm diameter 2.5mm")
+    (property "Sheetfile" "io_i2c.kicad_sch")
+    (property "Sheetname" "")
+    (attr through_hole)
+    (fp_text reference "R10" (at 5.109 -0.254 -90 unlocked) (layer "F.SilkS")
+      (effects (font (size 1 1) (thickness 0.15)))
+    )
+    (fp_text value "4.7k" (at -3.273 -0.254 -90 unlocked) (layer "F.SilkS")
+      (effects (font (size 1 1) (thickness 0.15)))
+    )
+    (fp_text user "${REFERENCE}" (at 1.27 -2.37 90) (layer "F.Fab")
+      (effects (font (size 1 1) (thickness 0.15)))
+    )
+    (fp_line (start 1.37 0) (end 1.44 0) (layer "F.SilkS") (width 0.12))
+    (fp_circle (center 0 0) (end 1.37 0) (layer "F.SilkS") (width 0.12) (fill none))
+    (fp_line (start -1.5 1.5) (end 3.59 1.5) (layer "F.CrtYd") (width 0.05))
+    (fp_line (start 3.59 1.5) (end 3.59 -1.5) (layer "F.CrtYd") (width 0.05))
+    (fp_line (start -1.5 -1.5) (end -1.5 1.5) (layer "F.CrtYd") (width 0.05))
+    (fp_line (start 3.59 -1.5) (end -1.5 -1.5) (layer "F.CrtYd") (width 0.05))
+    (fp_line (start 0 0) (end 2.54 0) (layer "F.Fab") (width 0.1))
+    (fp_circle (center 0 0) (end 1.25 0) (layer "F.Fab") (width 0.1) (fill none))
+    (pad "1" thru_hole circle locked (at 0 0 270) (size 1.6 1.6) (drill 0.8) (layers *.Cu *.Mask)
+      (net 3 "+5V") (pintype "passive"))
+    (pad "2" thru_hole oval locked (at 2.54 0 270) (size 1.6 1.6) (drill 0.8) (layers *.Cu *.Mask)
+      (net 91 "Net-(J5-Pad3)") (pintype "passive"))
+    (model "${KICAD6_3DMODEL_DIR}/Resistor_THT.3dshapes/R_Axial_DIN0207_L6.3mm_D2.5mm_P2.54mm_Vertical.wrl"
+      (offset (xyz 0 0 0))
+      (scale (xyz 1 1 1))
+      (rotate (xyz 0 0 0))
+    )
+  )
+  (footprint "Resistor_THT:R_Axial_DIN0207_L6.3mm_D2.5mm_P2.54mm_Vertical" (layer "F.Cu")
     (at 182.851 143.256)
     (descr "Resistor, Axial_DIN0207 series, Axial, Vertical, pin pitch=2.54mm, 0.25W = 1/4W, length*diameter=6.3*2.5mm^2, http://cdn-reichelt.de/documents/datenblatt/B400/1_4W%23YAG.pdf")
@@
       (effects (font (size 1 1) (thickness 0.15)))
     )
-    (fp_text value "74HCT74" (at 3.81 10.419 180) (layer "F.SilkS")
+    (fp_text value "74LS74" (at 3.81 10.419 180) (layer "F.SilkS")
       (effects (font (size 1 1) (thickness 0.15)))
     )
@@
       (effects (font (size 1 1) (thickness 0.15)))
     )
-    (fp_text value "74HCT138" (at 3.8 12.685 180) (layer "F.SilkS")
+    (fp_text value "74LS138" (at 3.8 12.685 180) (layer "F.SilkS")
       (effects (font (size 1 1) (thickness 0.15)))
     )
@@
       (effects (font (size 1 1) (thickness 0.15)))
     )
-    (fp_text value "74HCT125" (at 3.8 4.069 180) (layer "F.SilkS")
+    (fp_text value "74LS125" (at 3.8 4.069 180) (layer "F.SilkS")
       (effects (font (size 1 1) (thickness 0.15)))
     )
@@
   )
   (footprint "Resistor_THT:R_Axial_DIN0207_L6.3mm_D2.5mm_P2.54mm_Vertical" (layer "F.Cu")
-    (at 138.938 155.448 -90)
+    (at 139.192 155.673 -90)
     (descr "Resistor, Axial_DIN0207 series, Axial, Vertical, pin pitch=2.54mm, 0.25W = 1/4W, length*diameter=6.3*2.5mm^2, http://cdn-reichelt.de/documents/datenblatt/B400/1_4W%23YAG.pdf")
     (tags "Resistor Axial_DIN0207 series Axial Vertical pin pitch 2.54mm 0.25W = 1/4W length 6.3mm diameter 2.5mm")
@@
     (effects (font (size 0.5 0.5) (thickness 0.05)))
   )
-  (gr_text "Demon Debugger\nRev. D\nKnarfian Labs\nFrank Palazzolo\nEvan Allen" (at 115.824 138.938) (layer "F.SilkS")
+  (gr_text "Demon Debugger\nRev. E\nKnarfian Labs\nFrank Palazzolo\nEvan Allen" (at 115.824 138.938) (layer "F.SilkS")
     (effects (font (size 1 1) (thickness 0.15)))
   )
@@
   (segment (start 157.759 152.898) (end 157.739 152.918) (width 0.4) (layer "F.Cu") (net 3))
   (segment (start 111.64 152.908) (end 111.76 152.788) (width 0.4) (layer "F.Cu") (net 3))
+  (segment (start 132.827 152.918) (end 135.88 152.918) (width 0.4) (layer "F.Cu") (net 3))
   (segment (start 167.148031 154.697031) (end 165.349 152.898) (width 0.4) (layer "F.Cu") (net 3))
-  (segment (start 132.827 152.918) (end 139.089 152.918) (width 0.4) (layer "F.Cu") (net 3))
   (segment (start 108.458 152.908) (end 111.64 152.908) (width 0.4) (layer "F.Cu") (net 3))
   (segment (start 147.579 152.918) (end 148.778511 151.718489) (width 0.4) (layer "F.Cu") (net 3))
@@
   (segment (start 94.417511 151.708489) (end 88.455511 151.708489) (width 0.4) (layer "F.Cu") (net 3))
   (segment (start 146.379489 151.718489) (end 147.579 152.918) (width 0.4) (layer "F.Cu") (net 3))
+  (segment (start 135.89 155.673) (end 135.89 152.928) (width 0.4) (layer "F.Cu") (net 3))
   (segment (start 138.684 98.806) (end 159.512 98.806) (width 1) (layer "F.Cu") (net 3))
   (segment (start 151.318511 146.497511) (end 150.119 145.298) (width 0.4) (layer "F.Cu") (net 3))
@@
   (segment (start 153.999489 151.718489) (end 155.199 152.918) (width 0.4) (layer "F.Cu") (net 3))
   (segment (start 165.349 152.898) (end 157.759 152.898) (width 0.4) (layer "F.Cu") (net 3))
+  (segment (start 135.89 152.928) (end 135.88 152.918) (width 0.4) (layer "F.Cu") (net 3))
   (segment (start 156.539489 146.497511) (end 151.318511 146.497511) (width 0.4) (layer "F.Cu") (net 3))
   (segment (start 139.954 127.508) (end 141.224 126.238) (width 0.4) (layer "F.Cu") (net 3))
@@
   (segment (start 151.303511 151.718489) (end 153.999489 151.718489) (width 0.4) (layer "F.Cu") (net 3))
   (segment (start 105.664 98.806) (end 127.254 98.806) (width 1) (layer "F.Cu") (net 3))
+  (segment (start 135.88 152.918) (end 139.089 152.918) (width 0.4) (layer "F.Cu") (net 3))
   (segment (start 139.169 152.838) (end 140.288511 151.718489) (width 0.4) (layer "F.Cu") (net 3))
   (segment (start 183.896 153.028) (end 182.226969 154.697031) (width 0.4) (layer "F.Cu") (net 3))
@@
   (segment (start 116.387489 146.497511) (end 99.507511 146.497511) (width 0.4) (layer "F.Cu") (net 79))
   (segment (start 87.376 157.988) (end 90.678 157.988) (width 0.25) (layer "F.Cu") (net 80))
-  (segment (start 132.842 157.988) (end 138.938 157.988) (width 0.4) (layer "F.Cu") (net 80))
+  (segment (start 137.992489 159.412511) (end 139.192 158.213) (width 0.4) (layer "F.Cu") (net 80))
   (segment (start 93.218 157.988) (end 95.758 157.988) (width 0.25) (layer "F.Cu") (net 80))
+  (segment (start 134.266511 159.412511) (end 137.992489 159.412511) (width 0.4) (layer "F.Cu") (net 80))
   (segment (start 90.678 157.988) (end 93.218 157.988) (width 0.25) (layer "F.Cu") (net 80))
   (segment (start 95.758 157.988) (end 132.842 157.988) (width 0.25) (layer "F.Cu") (net 80))
   (segment (start 130.302 157.988) (end 132.842 157.988) (width 0.4) (layer "F.Cu") (net 80))
+  (segment (start 132.842 157.988) (end 134.266511 159.412511) (width 0.4) (layer "F.Cu") (net 80))
   (segment (start 127.254 112.268) (end 122.936 112.268) (width 0.4) (layer "F.Cu") (net 80))
   (via (at 122.936 112.268) (size 0.8) (drill 0.4) (layers "F.Cu" "B.Cu") (net 80))
@@
   (segment (start 175.509 163.571) (end 175.514 163.576) (width 0.4) (layer "B.Cu") (net 90))
   (segment (start 164.149489 151.449489) (end 154.826511 151.449489) (width 0.4) (layer "F.Cu") (net 91))
-  (segment (start 153.453511 150.076489) (end 96.811511 150.076489) (width 0.4) (layer "F.Cu") (net 91))
+  (segment (start 136.943511 150.076489) (end 96.811511 150.076489) (width 0.4) (layer "F.Cu") (net 91))
+  (segment (start 153.453511 150.076489) (end 136.943511 150.076489) (width 0.4) (layer "F.Cu") (net 91))
   (segment (start 154.826511 151.449489) (end 153.453511 150.076489) (width 0.4) (layer "F.Cu") (net 91))
+  (via (at 136.943511 150.076489) (size 0.8) (drill 0.4) (layers "F.Cu" "B.Cu") (net 91))
   (via (at 164.149489 151.449489) (size 0.8) (drill 0.4) (layers "F.Cu" "B.Cu") (net 91))
   (via (at 96.811511 150.076489) (size 0.8) (drill 0.4) (layers "F.Cu" "B.Cu") (net 91))
@@
   (segment (start 96.882511 150.147489) (end 96.882511 161.129511) (width 0.25) (layer "B.Cu") (net 91))
   (segment (start 164.149489 159.318489) (end 164.149489 151.449489) (width 0.4) (layer "B.Cu") (net 91))
+  (segment (start 137.089511 150.297511) (end 136.906 150.114) (width 0.4) (layer "B.Cu") (net 91))
+  (segment (start 135.89 158.213) (end 137.089511 157.013489) (width 0.4) (layer "B.Cu") (net 91))
   (segment (start 96.882511 161.129511) (end 100.345 164.592) (width 0.25) (layer "B.Cu") (net 91))
+  (segment (start 137.089511 157.013489) (end 137.089511 150.297511) (width 0.4) (layer "B.Cu") (net 91))
   (zone (net 1) (net_name "GND") (layers F&B.Cu) (hatch edge 0.508)
     (connect_pads (clearance 0.508))

Commit message: added CS multiplexer for use with rev E board, finished rev E layout
Parts:
- removed D10, D11, D12, D13, D14, D15, D16, D17, D18, D19, D3, D4, D5, D6, D7, D8, D9: 1N4148, Diode_THT:D_DO-35_SOD27_P2.54mm_Vertical_KathodeUp
- removed J7, J8: Conn_01x01, Connector_PinHeader_2.54mm:PinHeader_1x01_P2.54mm_Vertical
- removed R10, R2, R3, R9: 4.7k, Resistor_THT:R_Axial_DIN0207_L6.3mm_D2.5mm_P2.54mm_Vertical
- removed R7: 1k, Resistor_THT:R_Axial_DIN0207_L6.3mm_D2.5mm_P2.54mm_Vertical
- removed U3: 74LS125, Package_DIP:DIP-14_W7.62mm
- added C7: 0.1uF, Capacitor_THT:C_Axial_L3.8mm_D2.6mm_P7.50mm_Horizontal, F.Cu at (152.6, 164.3)
- added U5: 74LS04, Package_DIP:DIP-14_W7.62mm, F.Cu at (124.0, 143.0)
- added U8: 74LS30, Package_DIP:DIP-14_W7.62mm, F.Cu at (149.4, 156.7)
- added U9: 74LS257, Package_DIP:DIP-16_W7.62mm, F.Cu at (149.4, 143.0)
- J1: value extra CS -> read region
- J3: value Jumper Block -> Conn_01x01; footprint Connector_PinHeader_2.54mm:PinHeader_2x03_P2.54mm_Vertical -> Connector_PinHeader_2.54mm:PinHeader_1x01_P2.54mm_Vertical
- J5: value read region -> Conn_01x01; footprint Connector_PinHeader_2.54mm:PinHeader_1x03_P2.54mm_Vertical -> Connector_PinHeader_2.54mm:PinHeader_1x01_P2.54mm_Vertical
- U4: value 74LS138 -> 74LS02; footprint Package_DIP:DIP-16_W7.62mm -> Package_DIP:DIP-14_W7.62mm
- U7: value 74LS138 -> 74LS30; footprint Package_DIP:DIP-16_W7.62mm -> Package_DIP:DIP-14_W7.62mm
- moved J6 79.0 mm to (94.0, 163.6), turned to 0 degrees
- moved J3 76.1 mm to (96.0, 155.7), turned to 0 degrees
- moved J1 74.5 mm to (168.9, 161.8)
- moved R6 57.0 mm to (184.4, 127.0), turned to 90 degrees
- moved C3 55.7 mm to (128.3, 150.6), turned to 90 degrees
- moved C2 47.3 mm to (186.4, 150.6)
- moved C5 42.5 mm to (128.3, 164.3)
- moved C1 41.0 mm to (152.7, 150.6)
- moved U4 28.0 mm to (104.9, 143.0)
- moved G*** 26.3 mm to (156.2, 138.7)
- moved U2 25.5 mm to (183.1, 143.0)
- moved U7 19.3 mm to (124.0, 156.7)
- moved G*** 18.4 mm to (183.9, 156.5)
- moved J2 14.9 mm to (164.1, 145.5)
- moved J5 9.40 mm to (92.2, 155.7), turned to 0 degrees
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Connections:
- net /A7 renamed A7
- net /SDA renamed Net-(A1-Pad23)
- A1 pad 10: unconnected-(A1-Pad10) -> Target /OE
- A1 pad 22: /arduino control CS -> Target /CE
- A1 pad 5: /program OE -> unconnected-(A1-Pad5)
- A1 pad 7: /A8 -> A8
- A1 pad 8: /A9 -> A9
- A1 pad 9: /A10 -> A10
- J1 pad 1: Net-(J1-Pad1) -> GND
- J1 pad 2: /138 enable -> Net-(J1-Pad2)
- J1 pad 3: /target VPP -> +5V
- J16 pad 18: /Target CE -> Target /CE
- J16 pad 19: /A10 -> A10
- J16 pad 2: /A6 -> A6
- J16 pad 20: /Target OE -> Target /OE
- J16 pad 22: /A9 -> A9
- J16 pad 23: /A8 -> A8
- J16 pad 3: /A5 -> A5
- J2 pad 5: Net-(J2-Pad5) -> SDA
- J3 pad 1: /Target CE -> Net-(J3-Pad1)
- J4 pad 12: /A10 -> A10
- J4 pad 3: /A6 -> A6
- J4 pad 4: /A8 -> A8
- J4 pad 5: /A5 -> A5
- J4 pad 6: /A9 -> A9
- J5 pad 1: Net-(D18-Pad1) -> Net-(J3-Pad1)
- J6 pad 1: Net-(J6-Pad1) -> GND
- U1 pad 19: /A10 -> A10
- U1 pad 2: /A6 -> A6
- U1 pad 20: Net-(D10-Pad2) -> 2816/OE
- U1 pad 22: /A9 -> A9
- U1 pad 23: /A8 -> A8
- U1 pad 3: /A5 -> A5
- U1 pad 9: /D0 -> FLASHD0
- U2 pad 11: Net-(D16-Pad1) -> /WRITEARD
- U2 pad 3: Net-(D16-Pad1) -> /WRITEARD
- U4 pad 1: /A8 -> ROME
- U4 pad 10: Net-(D9-Pad1) -> Net-(U4-Pad10)
- U4 pad 11: Net-(D8-Pad1) -> Net-(U4-Pad11)
- U4 pad 14: Net-(D5-Pad1) -> +5V
- U4 pad 2: /A9 -> Target /OE
- U4 pad 3: /A10 -> Target /CE
- U4 pad 4: Net-(J3-Pad3) -> /READARD
- U4 pad 5: Net-(J3-Pad4) -> Net-(U4-Pad10)
- U4 pad 6: /138 enable -> Net-(U4-Pad10)
- U4 pad 7: Net-(U4-Pad7) -> GND
- U4 pad 8: GND -> Net-(J3-Pad1)
- U4 pad 9: Net-(D10-Pad1) -> Net-(J3-Pad1)
- U6 pad 20: /D0 -> FLASHD0
- U6 pad 8: /A5 -> A5
- U6 pad 9: /A6 -> A6
- U7 pad 1: /A5 -> +5V
- U7 pad 10: Net-(J5-Pad2) -> (no net)
- U7 pad 11: Net-(D15-Pad1) -> A10
- U7 pad 12: Net-(D14-Pad1) -> A9
- U7 pad 13: Net-(D13-Pad1) -> (no net)
- U7 pad 14: Net-(D12-Pad1) -> +5V
- U7 pad 2: /A6 -> ROME
- U7 pad 4: GND -> A6
- U7 pad 5: Net-(U4-Pad7) -> A8
- U7 pad 6: +5V -> Net-(U5-Pad8)
- U7 pad 7: Net-(D17-Pad1) -> GND
- U7 pad 8: GND -> Net-(U4-Pad11)
- U7 pad 9: Net-(D16-Pad1) -> (no net)
Routing:
- net A8: track 0.00 -> 208.3 mm, vias 0 -> 3
- net A10: track 0.00 -> 207.7 mm, vias 0 -> 3
- net A9: track 0.00 -> 202.6 mm, vias 0 -> 3
- net /A8: track 149.7 -> 0.00 mm, vias 3 -> 0
- net /A9: track 147.7 -> 0.00 mm, vias 3 -> 0
- net /A10: track 140.0 -> 0.00 mm, vias 2 -> 0
- net A5: track 0.00 -> 138.7 mm, vias 0 -> 3
- net Target /OE: track 0.00 -> 136.6 mm, vias 0 -> 3
- net Target /CE: track 0.00 -> 124.4 mm, vias 0 -> 3
- net A6: track 0.00 -> 122.6 mm, vias 0 -> 4
- net /A6: track 114.5 -> 0.00 mm, vias 2 -> 0
- net /Target OE: track 112.4 -> 0.00 mm, vias 2 -> 0
- net Net-(D10-Pad2): track 108.3 -> 0.00 mm, vias 1 -> 0
- net /A5: track 106.8 -> 0.00 mm, vias 2 -> 0
- net /Target CE: track 106.5 -> 0.00 mm, vias 2 -> 0
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Other:
- board text added: "Minimal interface is the arduino, Q1, R1, and R4 connected out J2"
- board text added: "U6, R5, C4, and fitting U1 with a 2816 enables onboard reprogramming of the flash chip"
- board text added: "cut here to insert read glitch snubber circuit"
- board text removed: "$000 $0FF"
- board text removed: "$100 $1FF"
- board text removed: "$200 $2FF"
- board text removed: "$300 $3FF"
- board text removed: "$400 $4FF"
- board text removed: "$500 $5FF"
- board text removed: "$600 $6FF"
- board text removed: "$700 $71F"
- board text removed: "$720 $73F"
- board text removed: "$740 $75F"
- board text removed: "$760 $77F"
- board text removed: "$780 $79F"
- board text removed: "$7A0 $7BF"
- board text removed: "$7C0 $7DF"
- board text removed: "$7E0 $7FF"
- board text removed: "1N4148"
- board text removed: "1N4148 or similar"
- board text removed: "4.7k"
- board text removed: "Active High"
- board text removed: "Active Low"
- board text removed: "CE"
- board text removed: "Ena"
- board text removed: "Extra CS on pin 21"
- board text removed: "From Arduino"
- board text removed: "In"
- board text removed: "Minimal interface is the arduino, Q1, R4, and R5 connected out J2"
- board text removed: "Normal Mode"
- board text removed: "OE"
- board text removed: "Out"
- board text removed: "U6, C4, and fitting U1 with a 2816 enables onboard reprogramming of the flash chip"

Commit message: added gerbers
Connections:
- J4 pad 10: /Target OE -> Target /OE
- J4 pad 14: /Target CE -> Target /CE
Changed lines of the file:
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@@
   (net 81 "unconnected-(U9-Pad14)")
   (net 82 "unconnected-(U9-Pad7)")
-  (net 83 "/Target OE")
-  (net 84 "unconnected-(A1-Pad5)")
-  (net 85 "/Target CE")
-  (net 86 "Net-(U5-Pad8)")
+  (net 83 "unconnected-(A1-Pad5)")
+  (net 84 "Net-(U5-Pad8)")
   (footprint "Capacitor_THT:C_Axial_L3.8mm_D2.6mm_P7.50mm_Horizontal" (layer "F.Cu")
     (at 128.27 150.562 90)
@@
       (net 2 "A8") (pintype "input"))
     (pad "6" thru_hole oval locked (at 0 12.7 270) (size 1.6 1.6) (drill 0.8) (layers *.Cu *.Mask)
-      (net 86 "Net-(U5-Pad8)") (pintype "input"))
+      (net 84 "Net-(U5-Pad8)") (pintype "input"))
     (pad "7" thru_hole oval locked (at 0 15.24 270) (size 1.6 1.6) (drill 0.8) (layers *.Cu *.Mask)
       (net 1 "GND") (pinfunction "GND") (pintype "power_in"))
@@
       (net 15 "/A3") (pinfunction "Pin_9") (pintype "passive"))
     (pad "10" thru_hole oval locked (at 2.54 10.16) (size 1.7 1.7) (drill 1) (layers *.Cu *.Mask)
-      (net 83 "/Target OE") (pinfunction "Pin_10") (pintype "passive"))
+      (net 11 "Target {slash}OE") (pinfunction "Pin_10") (pintype "passive"))
     (pad "11" thru_hole oval locked (at 0 12.7) (size 1.7 1.7) (drill 1) (layers *.Cu *.Mask)
       (net 13 "/A2") (pinfunction "Pin_11") (pintype "passive"))
@@
       (net 12 "/A1") (pinfunction "Pin_13") (pintype "passive"))
     (pad "14" thru_hole oval locked (at 2.54 15.24) (size 1.7 1.7) (drill 1) (layers *.Cu *.Mask)
-      (net 85 "/Target CE") (pinfunction "Pin_14") (pintype "passive"))
+      (net 19 "Target {slash}CE") (pinfunction "Pin_14") (pintype "passive"))
     (pad "15" thru_hole oval locked (at 0 17.78) (size 1.7 1.7) (drill 1) (layers *.Cu *.Mask)
       (net 10 "/A0") (pinfunction "Pin_15") (pintype "passive"))
@@
       (net 1 "GND") (pinfunction "GND") (pintype "power_in"))
     (pad "8" thru_hole oval locked (at 7.62 15.24 270) (size 1.6 1.6) (drill 0.8) (layers *.Cu *.Mask)
-      (net 86 "Net-(U5-Pad8)") (pintype "output"))
+      (net 84 "Net-(U5-Pad8)") (pintype "output"))
     (pad "9" thru_hole oval locked (at 7.62 12.7 270) (size 1.6 1.6) (drill 0.8) (layers *.Cu *.Mask)
       (net 58 "A5") (pintype "input"))
@@
       (net 1 "GND") (pinfunction "GND") (pintype "power_in"))
     (pad "5" thru_hole oval (at 0 10.16 180) (size 1.6 1.6) (drill 1) (layers *.Cu *.Mask)
-      (net 84 "unconnected-(A1-Pad5)") (pinfunction "D2") (pintype "bidirectional+no_connect"))
+      (net 83 "unconnected-(A1-Pad5)") (pinfunction "D2") (pintype "bidirectional+no_connect"))
     (pad "6" thru_hole oval (at 0 12.7 180) (size 1.6 1.6) (drill 1) (layers *.Cu *.Mask)
       (net 36 "/program WR") (pinfunction "D3") (pintype "bidirectional"))
@@
   (segment (start 145.612489 148.660489) (end 145.612489 155.518489) (width 0.4) (layer "B.Cu") (net 73))
   (segment (start 145.034 148.082) (end 145.612489 148.660489) (width 0.4) (layer "B.Cu") (net 73))
-  (segment (start 108.717 150.632) (end 108.717 154.188) (width 0.4) (layer "B.Cu") (net 86))
-  (segment (start 108.717 154.188) (end 111.257 156.728) (width 0.4) (layer "B.Cu") (net 86))
+  (segment (start 108.717 150.632) (end 108.717 154.188) (width 0.4) (layer "B.Cu") (net 84))
+  (segment (start 108.717 154.188) (end 111.257 156.728) (width 0.4) (layer "B.Cu") (net 84))
   (zone (net 1) (net_name "GND") (layers F&B.Cu) (hatch edge 0.508)
     (connect_pads (clearance 0.508))
